Commit message: added camera pose and corrected namespace error

File: deepleng_description_simplified/urdf/sensors.xacro (robot description, xacro)
@@ -32,6 +32,6 @@
   </xacro:default_imu> -->
   <!-- Mount a camera  -->
-  <xacro:default_camera namespace="${namespace}" parent_link="${namespace}/base_link" suffix="">
-    <origin xyz="0 0 0" rpy="0 0 0"/>
+  <xacro:default_camera namespace="${robot_namespace}" parent_link="${robot_namespace}/base_link" suffix="">
+    <origin xyz="1.35714 0 0 " rpy="1.57 0 0"/>
   </xacro:default_camera>
 </robot>

Commit message: fixed camera orientation

File: deepleng_description_simplified/urdf/sensors.xacro (robot description, xacro)
@@ -32,6 +32,7 @@
   </xacro:default_imu> -->
   <!-- Mount a camera  -->
+  <!-- wideangle_camera is the other option -->
   <xacro:default_camera namespace="${robot_namespace}" parent_link="${robot_namespace}/base_link" suffix="">
-    <origin xyz="1.35714 0 0 " rpy="1.57 0 0"/>
+    <origin xyz="1.35714 0 0 " rpy="0 0 0"/>
   </xacro:default_camera>
 </robot>
