Commit message: auv modelled with the diving cells as thrusters

File: deepleng_description_simplified/urdf/base.xacro (robot description, xacro)
@@ -20,11 +20,13 @@
   <xacro:property name="visual_mesh_file" value="file://$(find deepleng_description)/meshes/body.dae"/>
   <xacro:property name="visual_mesh_file_x_thruster" value="file://$(find deepleng_description)/meshes/x_thruster.dae"/>
-  <xacro:property name="visual_mesh_file_y_thruster_front" value="file://$(find deepleng_description)/meshes/y_thruster.dae"/>
-  <xacro:property name="visual_mesh_file_y_thruster_rear" value="file://$(find deepleng_description)/meshes/y_thruster.dae"/>
+  <xacro:property name="visual_mesh_file_y_thruster" value="file://$(find deepleng_description)/meshes/y_thruster.dae"/>
+  <!-- <xacro:property name="visual_mesh_file_y_thruster_rear" value="file://$(find deepleng_description)/meshes/y_thruster.dae"/> -->
+  <xacro:property name="visual_mesh_file_z_thruster" value="file://$(find deepleng_description)/meshes/z_thruster.dae"/>
    <!-- Collision geometry mesh -->
   <xacro:property name="collision_mesh_file" value="file://$(find deepleng_description)/meshes/body.stl"/>
   <xacro:property name="collision_mesh_file_x_thruster" value="file://$(find deepleng_description)/meshes/x_thruster.stl"/>
-  <xacro:property name="collision_mesh_file_y_thruster_front" value="file://$(find deepleng_description)/meshes/y_thruster.stl"/>
-  <xacro:property name="collision_mesh_file_y_thruster_rear" value="file://$(find deepleng_description)/meshes/y_thruster.stl"/>
+  <xacro:property name="collision_mesh_file_y_thruster" value="file://$(find deepleng_description)/meshes/y_thruster.stl"/>
+  <!-- <xacro:property name="collision_mesh_file_y_thruster_rear" value="file://$(find deepleng_description)/meshes/y_thruster.stl"/> -->
+  <xacro:property name="collision_mesh_file_z_thruster" value="file://$(find deepleng_description)/meshes/z_thruster.stl"/>
   <!-- <link name="dummy">
   </link> -->
@@ -87,5 +89,5 @@
           <origin xyz="0 0 0" rpy="0 0 0"/>
           <geometry>
-            <mesh filename="${visual_mesh_file_y_thruster_rear}" scale="1 1 1" />
+            <mesh filename="${visual_mesh_file_y_thruster}" scale="1 1 1" />
           </geometry>
         </visual>
@@ -93,5 +95,5 @@
           <origin xyz="0 0 0" rpy="0 0 0"/>
           <geometry>
-            <mesh filename="${collision_mesh_file_y_thruster_rear}" scale="1 1 1" />
+            <mesh filename="${collision_mesh_file_y_thruster}" scale="1 1 1" />
           </geometry>
         </collision>
@@ -109,5 +111,5 @@
           <origin xyz="0 0 0" rpy="0 0 0"/>
           <geometry>
-            <mesh filename="${visual_mesh_file_y_thruster_front}" scale="1 1 1" />
+            <mesh filename="${visual_mesh_file_y_thruster}" scale="1 1 1" />
           </geometry>
         </visual>
@@ -115,5 +117,49 @@
           <origin xyz="0 0 0" rpy="0 0 0"/>
           <geometry>
-            <mesh filename="${collision_mesh_file_y_thruster_front}" scale="1 1 1" />
+            <mesh filename="${collision_mesh_file_y_thruster}" scale="1 1 1" />
+          </geometry>
+        </collision>
+      </link>
+<!-- ================================================================================ -->
+      <link name="${robot_namespace}/diving_cell_front_link">
+        <inertial>
+          <mass value="0.01" />
+          <origin xyz="0.81495 0 0" rpy="0.0 0.0 0.0"/>
+          <inertia ixx="0.001" ixy="0" ixz="0"
+                   iyy="0.001" iyz="0"
+                   izz="0.001" />
+        </inertial>
+        <visual>
+          <origin xyz="0 0 0" rpy="0 0 0"/>
+          <geometry>
+            <mesh filename="${visual_mesh_file_z_thruster}" scale="1 1 1" />
+          </geometry>
+        </visual>
+        <collision>
+          <origin xyz="0 0 0" rpy="0 0 0"/>
+          <geometry>
+            <mesh filename="${collision_mesh_file_z_thruster}" scale="1 1 1" />
+          </geometry>
+        </collision>
+      </link>
+<!-- ================================================================================ -->
+      <link name="${robot_namespace}/diving_cell_rear_link">
+        <inertial>
+          <mass value="0.01" />
+          <origin xyz="-0.70343 0 0" rpy="0.0 0.0 0.0"/>
+          <inertia ixx="0.001" ixy="0" ixz="0"
+                   iyy="0.001" iyz="0"
+                   izz="0.001" />
+        </inertial>
+        <visual>
+          <origin xyz="0 0 0" rpy="0 0 0"/>
+          <geometry>
+            <mesh filename="${visual_mesh_file_z_thruster}" scale="1 1 1" />
+          </geometry>
+        </visual>
+        <collision>
+          <origin xyz="0 0 0" rpy="0 0 0"/>
+          <geometry>
+            <mesh filename="${collision_mesh_file_z_thruster}" scale="1 1 1" />
           </geometry>
         </collision>
@@ -142,4 +188,16 @@
         <axis xyz="0.0 1.0 0.0"/>
       </joint>
+      <joint name="diving_cell_front_joint" type="continuous">
+        <origin rpy="0.0 0.0 0.0" xyz="0.81495 0 0"/>
+        <parent link="${robot_namespace}/base_link"/>
+        <child link="${robot_namespace}/diving_cell_front_link"/>
+        <axis xyz="0.0 0.0 1.0"/>
+      </joint>
+      <joint name="diving_cell_rear_joint" type="continuous">
+        <origin rpy="0.0 0.0 0.0" xyz="-0.70343 0 0"/>
+        <parent link="${robot_namespace}/base_link"/>
+        <child link="${robot_namespace}/diving_cell_rear_link"/>
+        <axis xyz="0.0 0.0 1.0"/>
+      </joint>
 <!-- ================================================================================ -->
     <gazebo>
@@ -511,4 +569,251 @@
             </plugin>
     </gazebo>
+<!-- ================================================================================ -->
+    <gazebo>
+      <!-- Thruster ROS plugin -->
+      <plugin name="${robot_namespace}_z_thruster_front_model" filename="libuuv_thruster_ros_plugin.so">
+        <!-- Name of the thruster link -->
+        <linkName>${robot_namespace}/diving_cell_front_link</linkName>
+        <!-- Name of the joint between thruster and vehicle base link -->
+        <jointName>diving_cell_front_joint</jointName>
+        <!-- Make the thruster aware of its id -->
+        <thrusterID>4</thrusterID>
+        <!-- Gain of the input command signal -->
+        <gain>1</gain>
+              <!-- Maximum allowed input value for the input signal for thruster unit -->
+              <clampMax>60</clampMax>
+              <!-- Minimum allowed value for the input signal for thruster unit -->
+              <clampMin>-60</clampMin>
+              <!-- Minimum and maximum thrust force output allowed -->
+              <thrustMin>-60</thrustMin>
+              <thrustMax>60</thrustMax>
+              <!--
+              Value from 0 to 1 to set the efficiency of the output thrust force
+              Default value is 1.0
+              -->
+              <thrust_efficiency>1</thrust_efficiency>
+              <!--
+              Value from 0 to 1 to set the efficiency of the propeller as a factor
+              to be multiplied to the current value of the state variable at each
+              iteration.
+              Default value is 1.0
+              -->
+              <propeller_efficiency>1</propeller_efficiency>
+              <!--
+              Choose one of the propeller dynamics models below for your implementation
+              This will describe the dynamic model for the state variable of your thruster unit,
+              which can be, e.g., the angular velocity of the propeller.
+              -->
+              <!-- 1) Simple zero-order model -->
+              <dynamics>
+                <type>ZeroOrder</type>
+              </dynamics>
+              <!-- 2) First order model -->
+              <!--
+              <dynamics>
+                <type>FirstOrder</type>
+                <timeConstant>0.0</timeConstant>
+              </dynamics>
+            -->
+              <!-- 3) Yoerger's nonlinear dynamic model
+              For information on the model description:
+              [1] D. R. Yoerger, J. G. Cooke, and J.-J. E. Slotine, "The influence of
+                  thruster dynamics on underwater vehicle behavior and their incorporation
+                  into control system design," IEEE Journal of Oceanic Engineering, vol. 15,
+                  no. 3, pp. 167-178, Jul. 1990.
+              -->
+              <!--
+              <dynamics>
+                <type>Yoerger</type>
+                <alpha>0.0</alpha>
+                <beta>0.0</beta>
+              </dynamics>
+            -->
+              <!-- 4) Bessa's nonlinear dynamic model
+              For information on the model description:
+              [2] Bessa, Wallace Moreira, Max Suell Dutra, and Edwin Kreuzer. "Thruster
+                  dynamics compensation for the positioning of underwater robotic vehicles
+                  through a fuzzy sliding mode based approach." ABCM Symposium Series in
+                  Mechatronics. Vol. 2. 2006.
+              -->
+              <!--
+              <dynamics>
+                <type>Bessa</type>
+                <Jmsp>0.0</Jmsp>
+                <Kv1>0.0</Kv1>
+                <Kv2>0.0</Kv2>
+                <Kt>0.0</Kt>
+                <Rm>0.0</Rm>
+              </dynamics>
+            -->
+              <!--
+              Choose one of the model for the steady-state curve describing the
+              relationship between the state variable and the output thrust force
+              -->
+              <!-- 1) Basic curve
+              Input: x
+              Output: thrust
+              Function: thrust = rotorConstant * x * abs(x)
+              -->
+              <conversion>
+                <type>Basic</type>
+                <rotorConstant>0.01515</rotorConstant>
+              </conversion>
+              <!-- 2) Dead-zone nonlinearity described in Bessa, 2006
+              Input: x
+              Output: thrust
+              Function:
+              thrust = rotorConstantL * (x * abs(x) - deltaL), if x * abs(x) <= deltaL
+              thrust = 0, if deltaL < x * abs(x) < deltaR
+              thrust = rotorConstantR * (x * abs(x) - deltaR), if x * abs(x) >= deltaL
+              -->
+              <!--
+              <conversion>
+                <type>Bessa</type>
+                <rotorConstantL>0.0</rotorConstantL>
+                <rotorConstantR>0.0</rotorConstantR>
+                <deltaL>0.0</deltaL>
+                <deltaR>0.0</deltaR>
+              </conversion>
+            -->
+              <!-- 3) Linear interpolation
+              If you have access to the thruster's data sheet, for example,
+              you can enter samples of the curve's input and output values
+              and the thruster output will be found through linear interpolation
+              of the given samples.
+              -->
+              <!--
+              <conversion>
+                <type>LinearInterp</type>
+                <inputValues>0 1 2 3</inputValues>
+                <outputValues>0 1 2 3</outputValues>
+              </conversion>
+            -->
+            </plugin>
+    </gazebo>
+<!-- ================================================================================ -->
+    <gazebo>
+      <!-- Thruster ROS plugin -->
+      <plugin name="${robot_namespace}_z_thruster_rear_model" filename="libuuv_thruster_ros_plugin.so">
+        <!-- Name of the thruster link -->
+        <linkName>${robot_namespace}/diving_cell_rear_link</linkName>
+        <!-- Name of the joint between thruster and vehicle base link -->
+        <jointName>diving_cell_rear_joint</jointName>
+        <!-- Make the thruster aware of its id -->
+        <thrusterID>5</thrusterID>
+        <!-- Gain of the input command signal -->
+        <gain>1</gain>
+              <!-- Maximum allowed input value for the input signal for thruster unit -->
+              <clampMax>60</clampMax>
+              <!-- Minimum allowed value for the input signal for thruster unit -->
+              <clampMin>-60</clampMin>
+              <!-- Minimum and maximum thrust force output allowed -->
+              <thrustMin>-60</thrustMin>
+              <thrustMax>60</thrustMax>
+              <!--
+              Value from 0 to 1 to set the efficiency of the output thrust force
+              Default value is 1.0
+              -->
+              <thrust_efficiency>1</thrust_efficiency>
+              <!--
+              Value from 0 to 1 to set the efficiency of the propeller as a factor
+              to be multiplied to the current value of the state variable at each
+              iteration.
+              Default value is 1.0
+              -->
+              <propeller_efficiency>1</propeller_efficiency>
+              <!--
+              Choose one of the propeller dynamics models below for your implementation
+              This will describe the dynamic model for the state variable of your thruster unit,
+              which can be, e.g., the angular velocity of the propeller.
+              -->
+              <!-- 1) Simple zero-order model -->
+              <dynamics>
+                <type>ZeroOrder</type>
+              </dynamics>
+              <!-- 2) First order model -->
+              <!--
+              <dynamics>
+                <type>FirstOrder</type>
+                <timeConstant>0.0</timeConstant>
+              </dynamics>
+            -->
+              <!-- 3) Yoerger's nonlinear dynamic model
+              For information on the model description:
+              [1] D. R. Yoerger, J. G. Cooke, and J.-J. E. Slotine, "The influence of
+                  thruster dynamics on underwater vehicle behavior and their incorporation
+                  into control system design," IEEE Journal of Oceanic Engineering, vol. 15,
+                  no. 3, pp. 167-178, Jul. 1990.
+              -->
+              <!--
+              <dynamics>
+                <type>Yoerger</type>
+                <alpha>0.0</alpha>
+                <beta>0.0</beta>
+              </dynamics>
+            -->
+              <!-- 4) Bessa's nonlinear dynamic model
+              For information on the model description:
+              [2] Bessa, Wallace Moreira, Max Suell Dutra, and Edwin Kreuzer. "Thruster
+                  dynamics compensation for the positioning of underwater robotic vehicles
+                  through a fuzzy sliding mode based approach." ABCM Symposium Series in
+                  Mechatronics. Vol. 2. 2006.
+              -->
+              <!--
+              <dynamics>
+                <type>Bessa</type>
+                <Jmsp>0.0</Jmsp>
+                <Kv1>0.0</Kv1>
+                <Kv2>0.0</Kv2>
+                <Kt>0.0</Kt>
+                <Rm>0.0</Rm>
+              </dynamics>
+            -->
+              <!--
+              Choose one of the model for the steady-state curve describing the
+              relationship between the state variable and the output thrust force
+              -->
+              <!-- 1) Basic curve
+              Input: x
+              Output: thrust
+              Function: thrust = rotorConstant * x * abs(x)
+              -->
+              <conversion>
+                <type>Basic</type>
+                <rotorConstant>0.01515</rotorConstant>
+              </conversion>
+              <!-- 2) Dead-zone nonlinearity described in Bessa, 2006
+              Input: x
+              Output: thrust
+              Function:
+              thrust = rotorConstantL * (x * abs(x) - deltaL), if x * abs(x) <= deltaL
+              thrust = 0, if deltaL < x * abs(x) < deltaR
+              thrust = rotorConstantR * (x * abs(x) - deltaR), if x * abs(x) >= deltaL
+              -->
+              <!--
+              <conversion>
+                <type>Bessa</type>
+                <rotorConstantL>0.0</rotorConstantL>
+                <rotorConstantR>0.0</rotorConstantR>
+                <deltaL>0.0</deltaL>
+                <deltaR>0.0</deltaR>
+              </conversion>
+            -->
+              <!-- 3) Linear interpolation
+              If you have access to the thruster's data sheet, for example,
+              you can enter samples of the curve's input and output values
+              and the thruster output will be found through linear interpolation
+              of the given samples.
+              -->
+              <!--
+              <conversion>
+                <type>LinearInterp</type>
+                <inputValues>0 1 2 3</inputValues>
+                <outputValues>0 1 2 3</outputValues>
+              </conversion>
+            -->
+            </plugin>
+    </gazebo>
+<!-- ================================================================================ -->
     <gazebo reference="${robot_namespace}/base_link">
       <selfCollide>false</selfCollide>
@@ -521,4 +826,10 @@
     </gazebo>
     <gazebo reference="${robot_namespace}/y_thruster_front_link">
+      <selfCollide>false</selfCollide>
+    </gazebo>
+    <gazebo reference="${robot_namespace}/diving_cell_front_link">
+      <selfCollide>false</selfCollide>
+    </gazebo>
+    <gazebo reference="${robot_namespace}/diving_cell_rear_link">
       <selfCollide>false</selfCollide>
     </gazebo>

File: deepleng_description_simplified/urdf/sensors.xacro (robot description, xacro)
@@ -33,6 +33,6 @@
   <!-- Mount a camera  -->
   <!-- wideangle_camera is the other option -->
-  <xacro:default_camera namespace="${robot_namespace}" parent_link="${robot_namespace}/base_link" suffix="">
+  <xacro:wideangle_camera namespace="${robot_namespace}" parent_link="${robot_namespace}/base_link" suffix="">
     <origin xyz="1.35714 0 0 " rpy="0 0 0"/>
-  </xacro:default_camera>
+  </xacro:wideangle_camera>
 </robot>
