Commit message: fixed the camera configuration for a clear feed of the environment

File: uuv_sensor_plugins/uuv_sensor_ros_plugins/urdf/camera_snippets.xacro (robot description, xacro)
@@ -28,5 +28,5 @@
       parent_link="${parent_link}"
       topic="camera"
-      mass="0.01"
+      mass="0.1"
       update_rate="5"
       hfov="1.3962634"
@@ -113,5 +113,5 @@
           <clip>
             <near>0.02</near>
-            <far>300</far>
+            <far>3000</far>
           </clip>
           <noise>
@@ -143,5 +143,5 @@
   <xacro:macro name="underwater_camera_plugin_macro"
     params="namespace suffix parent_link topic mass update_rate
-      hfov width height stddev scale
+      hfov width height stddev
       *inertia *origin">
     <!-- Sensor link -->
@@ -154,5 +154,5 @@
       <visual>
         <geometry>
-          <mesh filename="file://$(find uuv_sensor_ros_plugins)/meshes/oe14-372.dae" scale="${scale} ${scale} ${scale}"/>
+          <mesh filename="file://$(find uuv_sensor_ros_plugins)/meshes/oe14-372.dae" scale="1 1 1"/>
         </geometry>
       </visual>
@@ -197,6 +197,6 @@
           </image>
           <clip>
-            <near>0.02</near>
-            <far>300</far>
+            <near>0.1</near>
+            <far>3000</far>
           </clip>
           <noise>

File: uuv_sensor_plugins/uuv_sensor_ros_plugins/urdf/camera_snippets_original.xacro (robot description, xacro)
@@ -28,10 +28,10 @@
       parent_link="${parent_link}"
       topic="camera"
-      mass="0.01"
-      update_rate="5"
-      hfov="1.3962634"
-      width="1360"
-      height="1024"
-      stddev="0.007"
+      mass="0.1"
+      update_rate="30"
+      hfov="1.5125"
+      width="768"
+      height="492"
+      stddev="0.02"
       scale="1.0">
       <inertia ixx="0.00001" ixy="0.0" ixz="0.0" iyy="0.00001" iyz="0.0" izz="0.00001" />
@@ -45,10 +45,10 @@
       parent_link="${parent_link}"
       topic="camera"
-      mass="0.01"
-      update_rate="5"
-      hfov="1.3962634"
-      width="1360"
-      height="1024"
-      stddev="0.007"
+      mass="0.015"
+      update_rate="30"
+      hfov="1.8125"
+      width="768"
+      height="492"
+      stddev="0.02"
       scale="1.0">
       <inertia ixx="0.00001" ixy="0.0" ixz="0.0" iyy="0.00001" iyz="0.0" izz="0.00001" />
@@ -112,6 +112,6 @@
           </image>
           <clip>
-            <near>0.02</near>
-            <far>300</far>
+            <near>0.05</near>
+            <far>3000</far>
           </clip>
           <noise>
@@ -143,5 +143,5 @@
   <xacro:macro name="underwater_camera_plugin_macro"
     params="namespace suffix parent_link topic mass update_rate
-      hfov width height stddev scale
+      hfov width height stddev
       *inertia *origin">
     <!-- Sensor link -->
@@ -154,5 +154,5 @@
       <visual>
         <geometry>
-          <mesh filename="file://$(find uuv_sensor_ros_plugins)/meshes/oe14-372.dae" scale="${scale} ${scale} ${scale}"/>
+          <mesh filename="file://$(find uuv_sensor_ros_plugins)/meshes/oe14-372.dae" scale="1 1 1"/>
         </geometry>
       </visual>
@@ -197,6 +197,6 @@
           </image>
           <clip>
-            <near>0.02</near>
-            <far>300</far>
+            <near>0.1</near>
+            <far>3000</far>
           </clip>
           <noise>
