Commit message: updated the deepeleng urdfs with the correct damping coefficients and base volume and fluid density

File: deepleng_description_gazebo7+ubuntu16/urdf/base.xacro (robot description, xacro)
@@ -12,9 +12,10 @@
     Vehicle's parameters (remember to enter the model parameters below)
   -->
-  <xacro:property name="mass" value="185.0"/> <!--eigentlich 115.957-->
+  <xacro:property name="mass" value="74.0"/>
   <!-- Center of gravity -->
-  <xacro:property name="cog" value="-0.05811 -0.00029 0.00492"/>
+  <xacro:property name="cog" value="0.0 0.0 -0.025"/>
   <!-- Fluid density -->
-  <xacro:property name="rho" value="1028"/>
+  <xacro:property name="rho" value="1000"/>
+<!--  <xacro:property name="rho" value="1028"/> for oceanic environments-->
     <!-- Visual mesh file for the vehicle -->
   <xacro:property name="visual_mesh_file" value="file://$(find deepleng_description)/meshes/body.dae"/>
@@ -213,7 +214,7 @@
         <gain>1</gain>
               <!-- Maximum allowed input value for the input signal for thruster unit -->
-              <clampMax>60</clampMax>
+              <clampMax>150</clampMax>
               <!-- Minimum allowed value for the input signal for thruster unit -->
-              <clampMin>-60</clampMin>
+              <clampMin>-150</clampMin>
               <!-- Minimum and maximum thrust force output allowed -->
               <thrustMin>-60</thrustMin>
@@ -289,5 +290,5 @@
               <conversion>
                 <type>Basic</type>
-                <rotorConstant>0.01515</rotorConstant>
+                <rotorConstant>0.00262</rotorConstant>
               </conversion>
               <!-- 2) Dead-zone nonlinearity described in Bessa, 2006
@@ -336,7 +337,7 @@
         <gain>1</gain>
               <!-- Maximum allowed input value for the input signal for thruster unit -->
-              <clampMax>60</clampMax>
+              <clampMax>150</clampMax>
               <!-- Minimum allowed value for the input signal for thruster unit -->
-              <clampMin>-60</clampMin>
+              <clampMin>-150</clampMin>
               <!-- Minimum and maximum thrust force output allowed -->
               <thrustMin>-60</thrustMin>
@@ -412,5 +413,5 @@
               <conversion>
                 <type>Basic</type>
-                <rotorConstant>0.01515</rotorConstant>
+                <rotorConstant>0.00262</rotorConstant>
               </conversion>
               <!-- 2) Dead-zone nonlinearity described in Bessa, 2006
@@ -459,7 +460,7 @@
         <gain>1</gain>
               <!-- Maximum allowed input value for the input signal for thruster unit -->
-              <clampMax>60</clampMax>
+              <clampMax>150</clampMax>
               <!-- Minimum allowed value for the input signal for thruster unit -->
-              <clampMin>-60</clampMin>
+              <clampMin>-150</clampMin>
               <!-- Minimum and maximum thrust force output allowed -->
               <thrustMin>-60</thrustMin>
@@ -535,5 +536,5 @@
               <conversion>
                 <type>Basic</type>
-                <rotorConstant>0.01515</rotorConstant>
+                <rotorConstant>0.00262</rotorConstant>
               </conversion>
               <!-- 2) Dead-zone nonlinearity described in Bessa, 2006
@@ -582,7 +583,7 @@
         <gain>1</gain>
               <!-- Maximum allowed input value for the input signal for thruster unit -->
-              <clampMax>60</clampMax>
+              <clampMax>150</clampMax>
               <!-- Minimum allowed value for the input signal for thruster unit -->
-              <clampMin>-60</clampMin>
+              <clampMin>-150</clampMin>
               <!-- Minimum and maximum thrust force output allowed -->
               <thrustMin>-60</thrustMin>
@@ -658,5 +659,5 @@
               <conversion>
                 <type>Basic</type>
-                <rotorConstant>0.01515</rotorConstant>
+                <rotorConstant>0.00262</rotorConstant>
               </conversion>
               <!-- 2) Dead-zone nonlinearity described in Bessa, 2006
@@ -705,7 +706,7 @@
         <gain>1</gain>
               <!-- Maximum allowed input value for the input signal for thruster unit -->
-              <clampMax>60</clampMax>
+              <clampMax>150</clampMax>
               <!-- Minimum allowed value for the input signal for thruster unit -->
-              <clampMin>-60</clampMin>
+              <clampMin>-150</clampMin>
               <!-- Minimum and maximum thrust force output allowed -->
               <thrustMin>-60</thrustMin>
@@ -781,5 +782,5 @@
               <conversion>
                 <type>Basic</type>
-                <rotorConstant>0.01515</rotorConstant>
+                <rotorConstant>0.00262</rotorConstant>
               </conversion>
               <!-- 2) Dead-zone nonlinearity described in Bessa, 2006

File: deepleng_description_gazebo7+ubuntu16/urdf/gazebo.xacro (robot description, xacro)
@@ -2,7 +2,8 @@
 <robot xmlns:xacro="http://www.ros.org/wiki/xacro">
     <!-- Center of buoyancy -->
-    <xacro:property name="deepleng_cob" value="0 0 0.1"/>
+    <xacro:property name="deepleng_cob" value="0 0 0.025"/>
     <!-- Vehicle's actual volume (Gazebo cannot compute the volume out of the mesh) -->
-    <xacro:property name="deepleng_volume" value="0.18"/>
+    <xacro:property name="deepleng_volume" value="0.074"/>
+<!--    <xacro:property name="deepleng_volume" value="0.071"/> if fluid density is 1028 -->
     <!-- Describing the dimensions of the vehicle's bounding box -->
     <xacro:property name="deepleng_length" value="3.0"/>
@@ -37,10 +38,10 @@
           <type>fossen</type>
           <added_mass>
-            100 0 0 0 0 0
-            0 100 0 0 0 0
-            0 0 100 0 0 0
-            0 0 0 100 0 0
-            0 0 0 0 100 0
-            0 0 0 0 0 100
+            70.5 0.0 0.0 0.0 0.0 0.0
+            0.0 478.72 0.0 0.0 0.0 0.0
+            0.0 0.0 478.72 0.0 0.0 0.0
+            0.0 0.0 0.0 0.07 0.0 0.0
+            0.0 0.0 0.0 0.0 368.15 0.0
+            0.0 0.0 0.0 0.0 0.0 368.15
           </added_mass>
           <!--
@@ -49,5 +50,10 @@
           -->
           <linear_damping>
-            -30 -80 -80 0 -200 -200
+            -15.51 0 0 0 0 0
+            0 -21.48 0 0 0 0
+            0 0 -21.48 0 0 0
+            0 0 0 -10.0 0 0
+            0 0 0 0 -32.0 0
+            0 0 0 0 0 -32.0
           </linear_damping>
           <!--
@@ -58,5 +64,10 @@
           -->
           <linear_damping_forward_speed>
-            -30 -80 -80 0 -200 -200
+            -15.51 0 0 0 0 0
+            0 -21.48 0 0 0 0
+            0 0 -21.48 0 0 0
+            0 0 0 -10.0 0 0
+            0 0 0 0 -32.0 0
+            0 0 0 0 0 -32.0
           </linear_damping_forward_speed>
           <!--
@@ -65,5 +76,10 @@
           -->
           <quadratic_damping>
-            -5 -300 -300 -15 -500 -500
+            -7.81 0 0 0 0 0
+            0 -779.4 0 0 0 0
+            0 0 -779.4 0 0 0
+            0 0 0 -15.0 0 0
+            0 0 0 0 -2020 0
+            0 0 0 0 0 -2020
           </quadratic_damping>
           <!--

File: deepleng_description_gazebo7+ubuntu16/urdf/snippets.xacro (robot description, xacro)
@@ -54,5 +54,5 @@
         <!-- Minimum allowed value for the input signal for thruster unit -->
         <clampMin>0</clampMin>
-        <!-- Minimum and maximum thrust force output allowed -->
+        <!-- Minimum and maximum thrust force output allowed -60 to 60-->
         <thrustMin>0</thrustMin>
         <thrustMax>10</thrustMax>
