Commit message: updated the deepleng discription to have the correct values for the hydrodynamic simulation

File: deepleng_description_gazebo9+ubuntu18/urdf/base.xacro (robot description, xacro)
@@ -12,9 +12,9 @@
     Vehicle's parameters (remember to enter the model parameters below)
   -->
-  <xacro:property name="mass" value="185.0"/>
+  <xacro:property name="mass" value="74.0"/>
   <!-- Center of gravity -->
-  <xacro:property name="cog" value="-0.05811 -0.00029 0.00492"/>
+  <xacro:property name="cog" value="0.0 0.0 -0.025"/>
   <!-- Fluid density -->
-  <xacro:property name="rho" value="1028"/>
+  <xacro:property name="rho" value="1000"/>
   <!--
     Visual mesh file for the vehicle, usually in DAE (Collada) format. Be sure to store the

File: deepleng_description_gazebo9+ubuntu18/urdf/gazebo.xacro (robot description, xacro)
@@ -2,7 +2,7 @@
 <robot xmlns:xacro="http://www.ros.org/wiki/xacro">
     <!-- Center of buoyancy -->
-    <xacro:property name="deepleng_cob" value="0 0 0.1"/>
+    <xacro:property name="deepleng_cob" value="0 0 0.025"/>
     <!-- Vehicle's actual volume (Gazebo cannot compute the volume out of the mesh) -->
-    <xacro:property name="deepleng_volume" value="0.18"/>
+    <xacro:property name="deepleng_volume" value="0.074"/>
     <!-- Describing the dimensions of the vehicle's bounding box -->
     <xacro:property name="deepleng_length" value="3.0"/>
@@ -40,10 +40,10 @@
           <type>fossen</type>
           <added_mass>
-            1     0     0     0     0     0
-            0     16    0     0     0     0
-            0     0     16    0     0     0
-            0     0     0     0.005 0     0
-            0     0     0     0     1.3   0
-            0     0     0     0     0     1.3
+            70.5  0.0  0.0  0.0  0.0  0.0
+            0.0  478.72  0.0  0.0  0.0  0.0
+            0.0  0.0  478.72  0.0  0.0  0.0
+            0.0  0.0  0.0  0.07  0.0  0.0
+            0.0  0.0  0.0  0.0  368.15  0.0
+            0.0  0.0  0.0  0.0  0.0  368.15
           </added_mass>
           <!--
@@ -52,6 +52,10 @@
           -->
           <linear_damping>
-            <!-- are these values correct ? -->
-            -30 -80 -80 0 -200 -200
+            -15.51  0  0  0  0  0
+            0  -21.48  0  0  0  0
+            0  0  -21.48  0  0  0
+            0  0  0  -10.0  0  0
+            0  0  0  0  -32.0  0
+            0  0  0  0  0  -32.0
           </linear_damping>
           <!--
@@ -62,5 +66,10 @@
           -->
           <linear_damping_forward_speed>
-            0 0 0 0 0 0
+            -15.51  0  0  0  0  0
+            0  -21.48  0  0  0  0
+            0  0  -21.48  0  0  0
+            0  0  0  -10.0  0  0
+            0  0  0  0  -32.0  0
+            0  0  0  0  0  -32.0
           </linear_damping_forward_speed>
           <!--
@@ -69,6 +78,10 @@
           -->
           <quadratic_damping>
-            <!-- are these values correct ? -->
-            -5 -300 -300 -15 -500 -500
+            -7.81  0  0  0  0  0
+            0  -779.4  0  0  0  0
+            0  0  -779.4  0  0  0
+            0  0  0  -15.0  0  0
+            0  0  0  0  -2020  0
+            0  0  0  0  0  -2020
           </quadratic_damping>
           <!--

File: deepleng_description_gazebo9+ubuntu18/urdf/snippets.xacro (robot description, xacro)
@@ -54,7 +54,7 @@
         <gain>1</gain>
         <!-- Maximum allowed input value for the input signal for thruster unit -->
-        <clampMax>60</clampMax>
+        <clampMax>150</clampMax>
         <!-- Minimum allowed value for the input signal for thruster unit -->
-        <clampMin>-60</clampMin>
+        <clampMin>-150</clampMin>
         <!-- Minimum and maximum thrust force output allowed -->
         <thrustMin>-60</thrustMin>
@@ -124,5 +124,5 @@
         <conversion>
           <type>Basic</type>
-          <rotorConstant>0.01515</rotorConstant>
+          <rotorConstant>0.00262</rotorConstant>
         </conversion>
         <!-- 2) Dead-zone nonlinearity described in Bessa, 2006
@@ -198,7 +198,7 @@
         <gain>1</gain>
         <!-- Maximum allowed input value for the input signal for thruster unit -->
-        <clampMax>60</clampMax>
+        <clampMax>150</clampMax>
         <!-- Minimum allowed value for the input signal for thruster unit -->
-        <clampMin>-60</clampMin>
+        <clampMin>-150</clampMin>
         <!-- Minimum and maximum thrust force output allowed -->
         <thrustMin>-60</thrustMin>
@@ -268,5 +268,5 @@
         <conversion>
           <type>Basic</type>
-          <rotorConstant>0.01515</rotorConstant>
+          <rotorConstant>0.00262</rotorConstant>
         </conversion>
         <!-- 2) Dead-zone nonlinearity described in Bessa, 2006
@@ -342,7 +342,7 @@
         <gain>1</gain>
         <!-- Maximum allowed input value for the input signal for thruster unit -->
-        <clampMax>60</clampMax>
+        <clampMax>150</clampMax>
         <!-- Minimum allowed value for the input signal for thruster unit -->
-        <clampMin>-60</clampMin>
+        <clampMin>-150</clampMin>
         <!-- Minimum and maximum thrust force output allowed -->
         <thrustMin>-60</thrustMin>
@@ -412,5 +412,5 @@
         <conversion>
           <type>Basic</type>
-          <rotorConstant>0.01515</rotorConstant>
+          <rotorConstant>0.00262</rotorConstant>
         </conversion>
         <!-- 2) Dead-zone nonlinearity described in Bessa, 2006
