Commit message: recalculated the values for the added mass matrix using the cylinder formula given in common.urdf.xacro in uuv_simulator package

File: deepleng_description_gazebo9+ubuntu18/urdf/gazebo.xacro (robot description, xacro)
@@ -2,5 +2,5 @@
 <robot xmlns:xacro="http://www.ros.org/wiki/xacro">
     <!-- Center of buoyancy -->
-    <xacro:property name="deepleng_cob" value="0 0 0.025"/>
+    <xacro:property name="deepleng_cob" value="0.0 0.0 0.025"/>
     <!-- Vehicle's actual volume (Gazebo cannot compute the volume out of the mesh) -->
     <xacro:property name="deepleng_volume" value="0.074"/>
@@ -35,15 +35,14 @@
         <!-- 1) Fossen's equation of motion -->
         <hydrodynamic_model>
-          <!-- values taken from  Light Autonomous Underwater Vehicle (LAUV), developed by the Laboratório de Sistemas e Tecnologia Subaquática (LSTS)
-          from Porto University and OceanScan-MST. Giving bad values can cause a crash in the simulation causing gazebo to close. As the linear or
+          <!-- values calculated for a cylinder using the formulas given in common.gazebo.xacro in the uuv_simulator package. Giving bad values can cause a crash in the simulation causing gazebo to close. As the linear or
           angular acceleration is calculated using these bad values can lead to division by zero resulting in nan values.-->
           <type>fossen</type>
           <added_mass>
-            70.5  0.0  0.0  0.0  0.0  0.0
-            0.0  478.72  0.0  0.0  0.0  0.0
-            0.0  0.0  478.72  0.0  0.0  0.0
-            0.0  0.0  0.0  0.07  0.0  0.0
-            0.0  0.0  0.0  0.0  368.15  0.0
-            0.0  0.0  0.0  0.0  0.0  368.15
+            7.4  0       0       0     0       0
+            0     184.72  0       0     0       0
+            0     0       184.72  0     0       0
+            0     0       0       0.07  0       0
+            0     0       0       0     46.18  0
+            0     0       0       0     0       46.18
           </added_mass>
           <!--
@@ -52,10 +51,5 @@
           -->
           <linear_damping>
-            -15.51  0  0  0  0  0
-            0  -21.48  0  0  0  0
-            0  0  -21.48  0  0  0
-            0  0  0  -10.0  0  0
-            0  0  0  0  -32.0  0
-            0  0  0  0  0  -32.0
+            -15.51 -21.48 -21.48 -10 -32 -32
           </linear_damping>
           <!--
@@ -66,10 +60,5 @@
           -->
           <linear_damping_forward_speed>
-            -15.51  0  0  0  0  0
-            0  -21.48  0  0  0  0
-            0  0  -21.48  0  0  0
-            0  0  0  -10.0  0  0
-            0  0  0  0  -32.0  0
-            0  0  0  0  0  -32.0
+            -15.51 -21.48 -21.48 -10 -32 -32
           </linear_damping_forward_speed>
           <!--
@@ -78,10 +67,5 @@
           -->
           <quadratic_damping>
-            -7.81  0  0  0  0  0
-            0  -779.4  0  0  0  0
-            0  0  -779.4  0  0  0
-            0  0  0  -15.0  0  0
-            0  0  0  0  -2020  0
-            0  0  0  0  0  -2020
+            -7.81 -779.4 -779.4 -15 -2020 -2020
           </quadratic_damping>
           <!--

File: deepleng_description_gazebo9+ubuntu18/urdf/snippets.xacro (robot description, xacro)
@@ -28,9 +28,9 @@
       </visual>
       <inertial>
-        <mass value="0.001" />
+        <mass value="0.01" />
         <origin xyz="0 0 0" rpy="0 0 0"/>
-        <inertia ixx="0.000000017" ixy="0.0" ixz="0.0"
-               iyy="0.000000017" iyz="0.0"
-               izz="0.000000017" />
+        <inertia ixx="0.001" ixy="0.0" ixz="0.0"
+               iyy="0.001" iyz="0.0"
+               izz="0.001" />
       </inertial>
     </link>
@@ -172,9 +172,9 @@
       </visual>
       <inertial>
-        <mass value="0.001" />
+        <mass value="0.01" />
         <origin xyz="0 0 0" rpy="0 0 0"/>
-        <inertia ixx="0.000000017" ixy="0.0" ixz="0.0"
-               iyy="0.000000017" iyz="0.0"
-               izz="0.000000017" />
+        <inertia ixx="0.001" ixy="0.0" ixz="0.0"
+               iyy="0.001" iyz="0.0"
+               izz="0.001" />
       </inertial>
     </link>
@@ -316,9 +316,9 @@
       </visual>
       <inertial>
-        <mass value="0.001" />
+        <mass value="0.01" />
         <origin xyz="0 0 0" rpy="0 0 0"/>
-        <inertia ixx="0.000000017" ixy="0.0" ixz="0.0"
-               iyy="0.000000017" iyz="0.0"
-               izz="0.000000017" />
+        <inertia ixx="0.001" ixy="0.0" ixz="0.0"
+               iyy="0.001" iyz="0.0"
+               izz="0.001" />
       </inertial>
     </link>
