Commit message: swapped the thruster ids for the z thrusters, rear thruster id=3 & front thruster id=4

File: deepleng_description_gazebo9+ubuntu18/urdf/actuators.xacro (robot description, xacro)
@@ -18,8 +18,8 @@
     </xacro:y_thruster_macro>
     <xacro:z_thruster_macro robot_namespace="${namespace}" thruster_id="3">
+        <origin xyz="-0.70343 0 0" rpy="0 0 0" />
+    </xacro:z_thruster_macro>
+    <xacro:z_thruster_macro robot_namespace="${namespace}" thruster_id="4">
         <origin xyz="0.81495 0 0" rpy="0 0 0" />
     </xacro:z_thruster_macro>
-    <xacro:z_thruster_macro robot_namespace="${namespace}" thruster_id="4">
-        <origin xyz="-0.70343 0 0" rpy="0 0 0" />
-    </xacro:z_thruster_macro>
 </robot>
